File: Level Shifter.kicad_pcb (KiCad board)
At the start: 2 copper layers, 36.6 x 27.9 mm, 15 parts, among them P1 3V3, P2 5V

Commit message: Gerbers tidied up
Parts:
- D1: value pwr -> PWR
- moved C1 1.05 mm to (163.1, 102.4)
- moved C2 0.97 mm to (176.3, 101.9)
Routing:
- net 3V3: track 17.1 -> 16.1 mm
Changed lines of the file:
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@@
     (thickness 1.6)
     (drawings 20)
-    (tracks 100)
+    (tracks 103)
     (zones 0)
     (modules 15)
@@
   )
   (module Capacitors_SMD:C_1206 placed (layer F.Cu)
-    (at 162.814 101.346 90)
+    (at 163.068 102.362 90)
     (descr "Capacitor SMD 1206, reflow soldering, AVX (see smccp.pdf)")
     (tags "capacitor 1206")
     (attr smd)
-    (fp_text reference C1 (at 0 -1.778 270) (layer F.SilkS)
-      (effects (font (size 0.7 0.7) (thickness 0.1)))
-    )
-    (fp_text value 0.1µF (at 0 1.778 90) (layer F.SilkS)
+    (fp_text reference C1 (at 2.794 0) (layer F.SilkS)
+      (effects (font (size 0.7 0.7) (thickness 0.1)))
+    )
+    (fp_text value 0.1µF (at 0.254 -2.032 90) (layer F.SilkS)
       (effects (font (size 0.7 0.7) (thickness 0.1)))
     )
@@
   )
   (module Capacitors_SMD:C_1206 placed (layer F.Cu)
-    (at 175.895 100.965)
+    (at 176.276 101.854)
     (descr "Capacitor SMD 1206, reflow soldering, AVX (see smccp.pdf)")
     (tags "capacitor 1206")
@@
       (effects (font (size 1 1) (thickness 0.15)))
     )
-    (fp_text value pwr (at -2.89814 0 180) (layer F.SilkS)
+    (fp_text value PWR (at -3.40614 0 180) (layer F.SilkS)
       (effects (font (size 1 1) (thickness 0.1)))
     )
@@
   )
   (gr_line (start 187.452 119.888) (end 187.452 91.948) (angle 90) (layer Edge.Cuts) (width 0.15))
-  (gr_text RTS (at 157.226 99.06) (layer F.SilkS)
+  (gr_text RTS (at 157.48 99.06) (layer F.SilkS)
     (effects (font (size 1.2 1.2) (thickness 0.2)))
   )
-  (gr_text RX (at 156.718 101.6) (layer F.SilkS)
+  (gr_text RX (at 156.972 101.6) (layer F.SilkS)
     (effects (font (size 1.2 1.2) (thickness 0.2)))
   )
@@
   )
   (gr_line (start 150.876 91.948) (end 150.876 119.888) (angle 90) (layer Edge.Cuts) (width 0.15))
-  (gr_text GND (at 157.48 111.76) (layer F.SilkS)
+  (gr_text GND (at 157.734 111.76) (layer F.SilkS)
     (effects (font (size 1.2 1.2) (thickness 0.2)))
   )
-  (gr_text CTS (at 157.226 109.22) (layer F.SilkS)
+  (gr_text CTS (at 157.48 109.22) (layer F.SilkS)
     (effects (font (size 1.2 1.2) (thickness 0.2)))
   )
-  (gr_text - (at 156.21 106.68) (layer F.SilkS)
+  (gr_text - (at 156.464 106.68) (layer F.SilkS)
     (effects (font (size 1.2 1.2) (thickness 0.2)))
   )
-  (gr_text TX (at 156.718 104.14) (layer F.SilkS)
+  (gr_text TX (at 156.972 104.14) (layer F.SilkS)
     (effects (font (size 1.2 1.2) (thickness 0.2)))
   )
@@
   (segment (start 167.32 104.73) (end 168.91 103.14) (width 0.381) (layer F.Cu) (net 1))
   (segment (start 166.214 104.73) (end 167.32 104.73) (width 0.381) (layer F.Cu) (net 1))
-  (segment (start 168.91 102.616) (end 168.91 101.219) (width 0.381) (layer F.Cu) (net 1))
+  (segment (start 168.91 101.727) (end 168.91 101.219) (width 0.381) (layer F.Cu) (net 1))
+  (segment (start 165.902 103.862) (end 166.214 104.174) (width 0.381) (layer F.Cu) (net 1))
   (segment (start 166.214 104.174) (end 166.214 104.73) (width 0.381) (layer F.Cu) (net 1))
-  (segment (start 164.886 102.846) (end 166.214 104.174) (width 0.381) (layer F.Cu) (net 1))
-  (segment (start 162.814 102.846) (end 164.886 102.846) (width 0.381) (layer F.Cu) (net 1))
-  (segment (start 168.91 101.727) (end 168.91 101.219) (width 0.381) (layer F.Cu) (net 1))
-  (segment (start 168.402 102.87) (end 168.91 101.727) (width 0.381) (layer F.Cu) (net 1))
-  (segment (start 162.814 102.846) (end 168.402 102.87) (width 0.381) (layer F.Cu) (net 1))
+  (segment (start 163.068 103.862) (end 165.902 103.862) (width 0.381) (layer F.Cu) (net 1))
+  (segment (start 167.41 103.862) (end 168.91 102.362) (width 0.381) (layer F.Cu) (net 1))
+  (segment (start 163.068 103.862) (end 167.41 103.862) (width 0.381) (layer F.Cu) (net 1))
+  (segment (start 168.91 102.362) (end 168.91 101.219) (width 0.381) (layer F.Cu) (net 1))
+  (segment (start 168.91 102.616) (end 168.91 102.362) (width 0.381) (layer F.Cu) (net 1))
   (segment (start 166.624 101.219) (end 166.624 98.171) (width 0.381) (layer F.Cu) (net 2))
   (segment (start 166.624 98.171) (end 167.005 97.79) (width 0.381) (layer F.Cu) (net 2))
@@
   (segment (start 176.784 113.538) (end 177.292 113.03) (width 0.381) (layer F.Cu) (net 2))
   (segment (start 176.784 114.374) (end 176.784 113.538) (width 0.381) (layer F.Cu) (net 2))
-  (via (at 178.816 99.822) (size 0.635) (drill 0.4) (layers F.Cu B.Cu) (net 2))
-  (segment (start 177.484437 100.137563) (end 177.395 100.965) (width 0.381) (layer F.Cu) (net 2))
-  (segment (start 178.816 99.822) (end 177.484437 100.137563) (width 0.381) (layer F.Cu) (net 2))
-  (segment (start 162.814 99.846) (end 164.592 98.552) (width 0.381) (layer F.Cu) (net 2))
-  (via (at 164.592 98.552) (size 0.635) (drill 0.4) (layers F.Cu B.Cu) (net 2))
+  (via (at 164.338 99.314) (size 0.635) (drill 0.4) (layers F.Cu B.Cu) (net 2))
+  (segment (start 163.068 100.584) (end 164.338 99.314) (width 0.381) (layer F.Cu) (net 2))
+  (segment (start 163.068 100.862) (end 163.068 100.584) (width 0.381) (layer F.Cu) (net 2))
+  (via (at 177.8 99.822) (size 0.635) (drill 0.4) (layers F.Cu B.Cu) (net 2))
+  (segment (start 177.776 99.846) (end 177.8 99.822) (width 0.381) (layer F.Cu) (net 2))
+  (segment (start 177.776 101.854) (end 177.776 99.846) (width 0.381) (layer F.Cu) (net 2))
   (segment (start 177.12 104.095) (end 177.165 104.14) (width 0.381) (layer F.Cu) (net 3))
   (segment (start 172.114 104.73) (end 170.098 104.73) (width 0.381) (layer F.Cu) (net 3))
@@
   (segment (start 171.196 103.632) (end 171.196 101.219) (width 0.381) (layer F.Cu) (net 3))
   (segment (start 174.395 102.146) (end 174.395 100.965) (width 0.381) (layer F.Cu) (net 3))
-  (segment (start 173.22 104.73) (end 174.395 103.555) (width 0.381) (layer F.Cu) (net 3))
-  (segment (start 174.395 103.555) (end 174.395 102.146) (width 0.381) (layer F.Cu) (net 3))
+  (segment (start 174.776 103.035) (end 174.776 101.854) (width 0.381) (layer F.Cu) (net 3))
+  (segment (start 174.776 103.174) (end 174.776 103.035) (width 0.381) (layer F.Cu) (net 3))
+  (segment (start 173.22 104.73) (end 174.776 103.174) (width 0.381) (layer F.Cu) (net 3))
   (segment (start 172.114 104.73) (end 173.22 104.73) (width 0.381) (layer F.Cu) (net 3))
   (segment (start 178.24772 97.32772) (end 178.308 97.388) (width 0.254) (layer F.Cu) (net 4))

Commit message: Revised with fixes
Parts:
- removed P1: 3V3, Pin_Headers:Pin_Header_Straight_1x06
- removed P2: 5V, Pin_Headers:Pin_Header_Straight_1x06
- removed the REF** at (162.6, 114.3)
- removed the REF** at (161.3, 95.8)
- removed TXB0104: TXB0104PW, Speculatrix_general:TSSOP-14_4.4x5mm_Pitch0.65mm_Pad0.35mm
- added IC1: TXB0104D_PW, Housings_SOIC:SOIC-14_3.9x8.7mm_Pitch1.27mm, F.Cu at (152.9, 59.2)
- added J1: 3V3, Pin_Headers:Pin_Header_Straight_1x06, F.Cu at (135.4, 55.4)
- added J2: 5V, Pin_Headers:Pin_Header_Straight_1x06, F.Cu at (173.7, 68.1)
- added J3: 3V3_test1, Pin_Headers:Pin_Header_Straight_1x03, F.Cu at (138.9, 55.4)
- added J4: 3V3_test2, Pin_Headers:Pin_Header_Straight_1x02, F.Cu at (138.9, 65.5)
- added J5: 5V_test, Pin_Headers:Pin_Header_Straight_1x06, F.Cu at (170.2, 68.1)
- added REF**: M3, Speculatrix_general:Mounting_hole_M3, F.Cu at (138.7, 73.5)
- added REF**: M3, Speculatrix_general:Mounting_hole_M3, F.Cu at (138.7, 46.5)
- added REF**: M3, Speculatrix_general:Mounting_hole_M3, F.Cu at (171.2, 46.5)
- added REF**: M3, Speculatrix_general:Mounting_hole_M3, F.Cu at (170.9, 73.7)
- D1: value PWR -> LED
- D2: value RX -> LED
- D3: value TX -> LED
- R3: value R3 -> 470
- R4: value R4 -> 470
- moved R2 52.0 mm to (159.5, 47.5)
- moved C1 51.4 mm to (146.8, 53.6)
- moved LM1 51.4 mm to (152.4, 49.3)
- moved C2 51.3 mm to (158.2, 53.8), turned to 90 degrees
- moved D3 51.2 mm to (162.3, 67.6)
- moved D2 50.1 mm to (159.0, 67.6)
- moved D1 49.7 mm to (163.3, 47.5)
- moved R1 48.7 mm to (154.2, 65.5), turned to 0 degrees
- moved R4 45.3 mm to (162.3, 72.9), turned to 270 degrees
- moved R3 44.2 mm to (159.0, 72.9), turned to 270 degrees
Connections:
- R1 pad 1: 5V -> 3V3
Routing:
- net /CTSH: track 12.7 -> 19.8 mm
- net /CTSL: track 12.6 -> 19.5 mm
- net /TXH: track 23.4 -> 29.1 mm
- net /TXL: track 12.9 -> 18.3 mm
- net 5V: track 11.9 -> 6.86 mm
- net /RTSH: track 14.3 -> 18.5 mm
- net /RXL: track 14.1 -> 18.1 mm
- net /RTSL: track 14.9 -> 18.3 mm
- net 3V3: track 16.1 -> 18.8 mm
- net GND: track 15.7 -> 18.3 mm, vias 7 -> 6
- net Net-(IC1-Pad8): track 3.71 -> 2.55 mm
- net /RXH: track 26.5 -> 27.6 mm, vias 4 -> 3
- net Net-(D2-Pad1): track 3.10 -> 2.46 mm
- net Net-(D3-Pad1): track 3.10 -> 2.46 mm
Other:
- board size 36.6 x 27.9 mm -> 44.1 x 36.8 mm
- net class Default: trace_width 0.254 -> 0.35; via_dia 0.635 -> 0.8; via_drill 0.381 -> 0.4
- net class power removed
- rule pad_to_mask_clearance: 0.2 -> 0
- board text added: "5V"
- board text added: "Machina Speculatrix Serial Level Shifter Rev 2.0"
- board text added: "—"
- board text removed: "+"
- board text removed: "+5V"
- board text removed: "-"
- board text removed: "Serial Level Shifter V2.0 https://bit.ly/speculatrix"
