File: Level Shifter.sch (KiCad schematic (older format))
At the start: 13 parts, among them IC1 TXB0104PW, P1 CONN_01X06, P2 5V_CONN

Commit message: Gerbers tidied up
Parts:
- D1: value Led_Small -> Led_PWR
- R2: value 330 -> 470
- R3, R4: value R -> 470
Other:
- moved on the sheet: D1, P2
Changed lines of the file:
@@
 L Level-Shifter-rescue:CONN_01X06-Level-Shifter-rescue P2
 U 1 1 5ADCD540
-P 7700 2150
-F 0 "P2" H 7700 2500 50  0000 C CNN
-F 1 "5V_CONN" V 7800 2150 50  0000 C CNN
-F 2 "Pin_Headers:Pin_Header_Straight_1x06" H 7700 2150 50  0001 C CNN
-F 3 "" H 7700 2150 50  0000 C CNN
-	1    7700 2150
+P 7675 2200
+F 0 "P2" H 7675 2550 50  0000 C CNN
+F 1 "5V_CONN" V 7775 2200 50  0000 C CNN
+F 2 "Pin_Headers:Pin_Header_Straight_1x06" H 7675 2200 50  0001 C CNN
+F 3 "" H 7675 2200 50  0000 C CNN
+	1    7675 2200
 	1    0    0    -1
 $EndComp
@@
 P 4500 2800
 F 0 "C1" H 4525 2900 50  0000 L CNN
-F 1 "0.1µF" H 4525 2700 50  0000 L CNN
+F 1 "0.1µF" H 4275 2700 50  0000 L CNN
 F 2 "Capacitors_SMD:C_1206" H 4538 2650 50  0001 C CNN
 F 3 "" H 4500 2800 50  0000 C CNN
@@
 	0    1    1    0
 $EndComp
-Text GLabel 6800 2400 0    50   Input ~ 0
-GND
-Text GLabel 4350 3100 0    50   Input ~ 0
-GND
 Text GLabel 4800 1250 0    50   Input ~ 0
 5V
@@
 Text GLabel 5650 1300 2    50   Input ~ 0
 3V3
-Text GLabel 6800 2200 0    50   Input ~ 0
+Text GLabel 6800 2250 0    50   Input ~ 0
 5V
 Text Label 6150 2350 0    50   ~ 0
@@
 TXH
 $Comp
-L power:PWR_FLAG #FLG01
-U 1 1 5ADCDBBD
-P 7450 2850
-F 0 "#FLG01" H 7450 2945 50  0001 C CNN
-F 1 "PWR_FLAG" H 7450 3030 50  0000 C CNN
-F 2 "" H 7450 2850 50  0000 C CNN
-F 3 "" H 7450 2850 50  0000 C CNN
-	1    7450 2850
-	0    1    1    0
-$EndComp
-$Comp
 L power:PWR_FLAG #FLG02
 U 1 1 5ADCDBDF
-P 7675 2600
-F 0 "#FLG02" H 7675 2695 50  0001 C CNN
-F 1 "PWR_FLAG" H 7675 2780 50  0000 C CNN
-F 2 "" H 7675 2600 50  0000 C CNN
-F 3 "" H 7675 2600 50  0000 C CNN
-	1    7675 2600
+P 7475 1575
+F 0 "#FLG02" H 7475 1670 50  0001 C CNN
+F 1 "PWR_FLAG" H 7475 1755 50  0000 C CNN
+F 2 "" H 7475 1575 50  0000 C CNN
+F 3 "" H 7475 1575 50  0000 C CNN
+	1    7475 1575
 	0    1    1    0
 $EndComp
@@
 GND
 NoConn ~ 3800 2250
-Text Label 4000 2350 2    50   ~ 0
+Text Label 3850 2350 0    50   ~ 0
 CTSL
-Text Label 4075 2050 2    50   ~ 0
+Text Label 3850 2050 0    50   ~ 0
 RXL
-Text Label 4075 2150 2    50   ~ 0
+Text Label 3850 2150 0    50   ~ 0
 TXL
-Text Label 4075 1950 2    50   ~ 0
+Text Label 3850 1950 0    50   ~ 0
 RTSL
 Wire Wire Line
@@
 	4500 2950 4500 3100
 Wire Wire Line
-	4350 3100 4500 3100
-Wire Wire Line
 	5800 1900 5900 1900
 Wire Wire Line
@@
 Wire Wire Line
 	5900 3100 5900 3000
-Connection ~ 4500 3100
 Wire Wire Line
 	4750 2600 4700 2600
@@
 L Level-Shifter-rescue:Led_Small-Level-Shifter-rescue D1
 U 1 1 5ADD89E2
-P 6900 2775
-F 0 "D1" H 6850 2900 50  0000 L CNN
-F 1 "Led_Small" H 6725 2675 50  0000 L CNN
-F 2 "LEDs:LED_1206" V 6900 2775 50  0001 C CNN
-F 3 "" V 6900 2775 50  0000 C CNN
-	1    6900 2775
+P 6900 2675
+F 0 "D1" H 6850 2800 50  0000 L CNN
+F 1 "Led_PWR" H 6725 2575 50  0000 L CNN
+F 2 "LEDs:LED_1206" V 6900 2675 50  0001 C CNN
+F 3 "" V 6900 2675 50  0000 C CNN
+	1    6900 2675
 	0    -1   -1   0
 $EndComp
@@
 P 6650 3100
 F 0 "R2" V 6730 3100 50  0000 C CNN
-F 1 "330" V 6650 3100 50  0000 C CNN
+F 1 "470" V 6650 3100 50  0000 C CNN
 F 2 "Resistors_SMD:R_1206" V 6580 3100 50  0001 C CNN
 F 3 "" H 6650 3100 50  0000 C CNN
@@
 $EndComp
 Wire Wire Line
-	6900 2750 6900 2875
+	6900 2750 6900 2775
 Wire Wire Line
 	6900 3100 6800 3100
@@
 P 7300 3650
 F 0 "R4" V 7380 3650 50  0000 C CNN
-F 1 "R" V 7300 3650 50  0000 C CNN
+F 1 "470" V 7300 3650 50  0000 C CNN
 F 2 "Resistors_SMD:R_1206" V 7230 3650 50  0001 C CNN
 F 3 "" H 7300 3650 50  0000 C CNN
@@
 P 7100 3650
 F 0 "R3" V 7180 3650 50  0000 C CNN
-F 1 "R" V 7100 3650 50  0000 C CNN
+F 1 "470" V 7100 3650 50  0000 C CNN
 F 2 "Resistors_SMD:R_1206" V 7030 3650 50  0001 C CNN
 F 3 "" H 7100 3650 50  0000 C CNN
@@
 Wire Wire Line
 	7200 3900 7300 3900
-Connection ~ 6900 2875
-Wire Wire Line
-	6900 2875 6900 3100
-Wire Wire Line
-	6800 2200 6900 2200
-Wire Wire Line
-	6900 2675 6900 2200
-Connection ~ 6900 2200
-Wire Wire Line
-	6900 2200 7250 2200
-Wire Wire Line
-	6800 2400 7150 2400
-Wire Wire Line
-	7450 2850 7150 2850
-Wire Wire Line
-	7150 2850 7150 2400
-Connection ~ 7150 2400
-Wire Wire Line
-	7150 2400 7500 2400
-Wire Wire Line
-	7675 2600 7250 2600
-Wire Wire Line
-	7250 2600 7250 2200
-Connection ~ 7250 2200
-Wire Wire Line
-	7250 2200 7500 2200
-Wire Wire Line
-	7500 2100 7300 2100
-Wire Wire Line
-	6475 2100 6475 2250
-Wire Wire Line
-	6475 2250 5800 2250
-Wire Wire Line
-	7500 2000 7100 2000
-Wire Wire Line
-	6425 2000 6425 2150
-Wire Wire Line
-	6425 2150 5800 2150
-Wire Wire Line
-	7500 1900 6375 1900
-Wire Wire Line
-	6375 1900 6375 2050
+Connection ~ 6900 2775
+Wire Wire Line
+	6900 2775 6900 3100
+Wire Wire Line
+	6800 2250 6900 2250
+Wire Wire Line
+	6900 2575 6900 2250
+Connection ~ 6900 2250
+Wire Wire Line
+	6900 2250 7225 2250
+Wire Wire Line
+	7475 1575 7225 1575
+Wire Wire Line
+	7225 1575 7225 2250
+Connection ~ 7225 2250
+Wire Wire Line
+	7225 2250 7475 2250
+Wire Wire Line
+	7475 2150 7300 2150
+Wire Wire Line
+	6525 2150 6525 2250
+Wire Wire Line
+	6525 2250 5800 2250
+Wire Wire Line
+	7475 2050 7100 2050
+Wire Wire Line
+	6450 2050 6450 2150
+Wire Wire Line
+	6450 2150 5800 2150
+Wire Wire Line
+	7475 1950 6375 1950
+Wire Wire Line
+	6375 1950 6375 2050
 Wire Wire Line
 	6375 2050 5800 2050
 Wire Wire Line
-	7300 3200 7300 2100
-Connection ~ 7300 2100
-Wire Wire Line
-	6475 2100 7300 2100
-Wire Wire Line
-	7100 2950 7100 2000
-Connection ~ 7100 2000
-Wire Wire Line
-	7100 2000 6425 2000
+	7300 3200 7300 2150
+Connection ~ 7300 2150
+Wire Wire Line
+	6525 2150 7300 2150
+Wire Wire Line
+	7100 2950 7100 2050
+Connection ~ 7100 2050
+Wire Wire Line
+	7100 2050 6450 2050
 Wire Wire Line
 	3800 2350 4750 2350
 Wire Wire Line
-	7500 2300 6500 2300
-Wire Wire Line
-	6500 2300 6500 2350
-Wire Wire Line
-	6500 2350 5800 2350
-Wire Wire Line
-	4750 2050 4175 2050
-Wire Wire Line
-	4175 2050 4175 1950
-Wire Wire Line
-	4175 1950 3800 1950
-Wire Wire Line
-	4750 2150 4150 2150
-Wire Wire Line
-	4150 2150 4150 2050
-Wire Wire Line
-	4150 2050 3800 2050
-Wire Wire Line
-	4750 2250 4125 2250
-Wire Wire Line
-	4125 2250 4125 2150
-Wire Wire Line
-	4125 2150 3800 2150
+	4750 2050 4150 2050
+Wire Wire Line
+	4150 2050 4150 1950
+Wire Wire Line
+	4150 1950 3800 1950
+Wire Wire Line
+	4750 2150 4100 2150
+Wire Wire Line
+	4100 2150 4100 2050
+Wire Wire Line
+	4100 2050 3800 2050
+Wire Wire Line
+	4750 2250 4050 2250
+Wire Wire Line
+	4050 2250 4050 2150
+Wire Wire Line
+	4050 2150 3800 2150
+Wire Wire Line
+	5800 2350 7475 2350
+$Comp
+L power:GND #PWR0101
+U 1 1 5CFB243D
+P 7475 2800
+F 0 "#PWR0101" H 7475 2550 50  0001 C CNN
+F 1 "GND" H 7475 2650 50  0000 C CNN
+F 2 "" H 7475 2800 50  0000 C CNN
+F 3 "" H 7475 2800 50  0000 C CNN
+	1    7475 2800
+	1    0    0    -1
+$EndComp
+Wire Wire Line
+	7475 2450 7475 2675
+$Comp
+L power:PWR_FLAG #FLG0101
+U 1 1 5CFB7978
+P 7600 2675
+F 0 "#FLG0101" H 7600 2750 50  0001 C CNN
+F 1 "PWR_FLAG" V 7600 2803 50  0000 L CNN
+F 2 "" H 7600 2675 50  0001 C CNN
+F 3 "~" H 7600 2675 50  0001 C CNN
+	1    7600 2675
+	0    1    1    0
+$EndComp
+Wire Wire Line
+	7600 2675 7475 2675
+Connection ~ 7475 2675
+Wire Wire Line
+	7475 2675 7475 2800
+$Comp
+L power:GND #PWR0102
+U 1 1 5CFB9AF2
+P 4500 3275
+F 0 "#PWR0102" H 4500 3025 50  0001 C CNN
+F 1 "GND" H 4500 3125 50  0000 C CNN
+F 2 "" H 4500 3275 50  0000 C CNN
+F 3 "" H 4500 3275 50  0000 C CNN
+	1    4500 3275
+	1    0    0    -1
+$EndComp
+Wire Wire Line
+	4500 3275 4500 3100
+Connection ~ 4500 3100
 $EndSCHEMATC

Commit message: Revised with fixes
Parts:
- removed D1: Led_PWR, LEDs:LED_1206, symbol Level-Shifter-rescue:Led_Small-Level-Shifter-rescue
- removed D2: Led_RX, LEDs:LED_1206, symbol Level-Shifter-rescue:Led_Small-Level-Shifter-rescue
- removed D3: Led_TX, LEDs:LED_1206, symbol Level-Shifter-rescue:Led_Small-Level-Shifter-rescue
- removed IC1: TXB0104PW, Speculatrix_general:TSSOP-14_4.4x5mm_Pitch0.65mm_Pad0.35mm, symbol speculatrix_power:TXB0104PW
- removed P1: CONN_01X06, Pin_Headers:Pin_Header_Straight_1x06, symbol Level-Shifter-rescue:CONN_01X06-Level-Shifter-rescue
- removed P2: 5V_CONN, Pin_Headers:Pin_Header_Straight_1x06, symbol Level-Shifter-rescue:CONN_01X06-Level-Shifter-rescue
- added D1, D2, D3: LED, LEDs:LED_1206, symbol Device:LED
- added IC1: TXB0104D_PW, Housings_SOIC:SOIC-14_3.9x8.7mm_Pitch1.27mm, symbol speculatrix_power:TXB0104D_PW
- added J1: 3V3, Pin_Headers:Pin_Header_Straight_1x06, symbol Connector:Conn_01x06_Male
- added J2: 5V, Pin_Headers:Pin_Header_Straight_1x06, symbol Connector:Conn_01x06_Male
- added J3: 3V3_test1, Pin_Headers:Pin_Header_Straight_1x03, symbol Connector:Conn_01x03_Male
- added J4: 3V3_test2, Pin_Headers:Pin_Header_Straight_1x02, symbol Connector:Conn_01x02_Male
- added J5: 5V_test, Pin_Headers:Pin_Header_Straight_1x06, symbol Connector:Conn_01x06_Male
Connections:
- net 3V3: now also R1.1, IC1.1 (VCCA)
- net 5V: now also D1.2 (A), IC1.14 (VCCB), J2.3 (Pin_3), J5.3 (Pin_3); no longer R1.1
- net CTSH: now also IC1.10 (B4), J2.2 (Pin_2), J5.2 (Pin_2)
- net CTSL: now also IC1.5 (A4), J1.5 (Pin_5), J4.1 (Pin_1)
- net GND: now also IC1.7 (GND), J1.6 (Pin_6), J2.1 (Pin_1), J4.2 (Pin_2), J5.1 (Pin_1)
- net RTSH: now also IC1.13 (B1), J2.6 (Pin_6), J5.6 (Pin_6)
- net RTSL: now also IC1.2 (A1), J1.1 (Pin_1), J3.1 (Pin_1)
- net RXH: now also D2.2 (A), IC1.12 (B2), J2.5 (Pin_5), J5.5 (Pin_5)
- net RXL: now also IC1.3 (A2), J1.2 (Pin_2), J3.2 (Pin_2)
- net TXH: now also D3.2 (A), IC1.11 (B3), J2.4 (Pin_4), J5.4 (Pin_4)
- net TXL: now also IC1.4 (A3), J1.3 (Pin_3), J3.3 (Pin_3)
- net at R1.2: now also IC1.8 (OE)
- net at R2.1: now also D1.1 (K)
- net at R4.1: now also D3.1 (K)
- net at R3.1: now also D2.1 (K)
Changed lines of the file:
@@
 Sheet 1 1
 Title "Serial Comms Level Shifter"
-Date "2019-06-06"
-Rev "1.1"
+Date "2019-07-22"
+Rev "2.0"
 Comp "https://mansfield-devine.com/speculatrix/"
 Comment1 "Intended for use with SmartParallel board."
@@
 Comment4 ""
 $EndDescr
-$Comp
-L Level-Shifter-rescue:CONN_01X06-Level-Shifter-rescue P2
-U 1 1 5ADCD540
-P 7675 2200
-F 0 "P2" H 7675 2550 50  0000 C CNN
-F 1 "5V_CONN" V 7775 2200 50  0000 C CNN
-F 2 "Pin_Headers:Pin_Header_Straight_1x06" H 7675 2200 50  0001 C CNN
-F 3 "" H 7675 2200 50  0000 C CNN
-	1    7675 2200
-	1    0    0    -1
-$EndComp
-$Comp
-L speculatrix_power:LM1117 LM1
-U 1 1 5ADCD5C1
-P 5300 1450
-F 0 "LM1" H 5250 1750 60  0000 C CNN
-F 1 "LM1117" H 5250 1400 60  0000 C CNN
-F 2 "TO_SOT_Packages_SMD:SOT-223" H 5300 1450 60  0001 C CNN
-F 3 "" H 5300 1450 60  0000 C CNN
-	1    5300 1450
-	1    0    0    -1
-$EndComp
-$Comp
-L speculatrix_power:TXB0104PW IC1
-U 1 1 5ADCD97A
-P 5300 2350
-F 0 "IC1" H 5300 2950 60  0000 C CNN
-F 1 "TXB0104PW" H 5300 1950 60  0000 C CNN
-F 2 "Speculatrix_general:TSSOP-14_4.4x5mm_Pitch0.65mm_Pad0.35mm" H 5550 1950 60  0001 C CNN
-F 3 "" H 5550 1950 60  0000 C CNN
-	1    5300 2350
-	1    0    0    -1
-$EndComp
 $Comp
 L Device:C C2
@@
 5V
 Text GLabel 6400 2600 2    50   Input ~ 0
-5V
+3V3
 Wire Wire Line
 	5800 2600 5950 2600
 Wire Wire Line
 	6250 2600 6400 2600
-$Comp
-L Level-Shifter-rescue:CONN_01X06-Level-Shifter-rescue P1
-U 1 1 5ADCDD74
-P 3600 2200
-F 0 "P1" H 3600 2550 50  0000 C CNN
-F 1 "CONN_01X06" V 3700 2200 50  0000 C CNN
-F 2 "Pin_Headers:Pin_Header_Straight_1x06" H 3600 2200 50  0001 C CNN
-F 3 "" H 3600 2200 50  0000 C CNN
-	1    3600 2200
-	-1   0    0    1
-$EndComp
 Text GLabel 4400 1900 0    50   Input ~ 0
 3V3
 Text GLabel 3800 2450 2    50   Input ~ 0
 GND
-NoConn ~ 3800 2250
+NoConn ~ 3050 2250
 Text Label 3850 2350 0    50   ~ 0
 CTSL
@@
 	4700 2600 4700 3100
 Connection ~ 4700 3100
-$Comp
-L Level-Shifter-rescue:Led_Small-Level-Shifter-rescue D1
-U 1 1 5ADD89E2
-P 6900 2675
-F 0 "D1" H 6850 2800 50  0000 L CNN
-F 1 "Led_PWR" H 6725 2575 50  0000 L CNN
-F 2 "LEDs:LED_1206" V 6900 2675 50  0001 C CNN
-F 3 "" V 6900 2675 50  0000 C CNN
-	1    6900 2675
-	0    -1   -1   0
-$EndComp
 $Comp
 L Device:R R2
@@
 $EndComp
 Wire Wire Line
-	6900 2750 6900 2775
-Wire Wire Line
 	6900 3100 6800 3100
 Connection ~ 5900 3100
-$Comp
-L Level-Shifter-rescue:Led_Small-Level-Shifter-rescue D3
-U 1 1 5AF92CC9
-P 7300 3300
-F 0 "D3" H 7250 3425 50  0000 L CNN
-F 1 "Led_TX" H 7125 3200 50  0000 L CNN
-F 2 "LEDs:LED_1206" V 7300 3300 50  0001 C CNN
-F 3 "" V 7300 3300 50  0000 C CNN
-	1    7300 3300
-	0    -1   -1   0
-$EndComp
-$Comp
-L Level-Shifter-rescue:Led_Small-Level-Shifter-rescue D2
-U 1 1 5AF92D13
-P 7100 3050
-F 0 "D2" H 7050 3175 50  0000 L CNN
-F 1 "Led_RX" H 6925 2950 50  0000 L CNN
-F 2 "LEDs:LED_1206" V 7100 3050 50  0001 C CNN
-F 3 "" V 7100 3050 50  0000 C CNN
-	1    7100 3050
-	0    -1   -1   0
-$EndComp
 $Comp
 L Device:R R4
@@
 $EndComp
 Wire Wire Line
-	7300 3500 7300 3400
-Wire Wire Line
-	7100 3500 7100 3150
+	7300 3500 7300 3250
+Wire Wire Line
+	7100 3500 7100 3250
 Wire Wire Line
 	7300 3900 7300 3800
@@
 Wire Wire Line
 	7200 3900 7300 3900
-Connection ~ 6900 2775
-Wire Wire Line
-	6900 2775 6900 3100
 Wire Wire Line
 	6800 2250 6900 2250
@@
 Connection ~ 7225 2250
 Wire Wire Line
-	7225 2250 7475 2250
-Wire Wire Line
-	7475 2150 7300 2150
-Wire Wire Line
 	6525 2150 6525 2250
 Wire Wire Line
 	6525 2250 5800 2250
 Wire Wire Line
-	7475 2050 7100 2050
-Wire Wire Line
 	6450 2050 6450 2150
 Wire Wire Line
 	6450 2150 5800 2150
 Wire Wire Line
-	7475 1950 6375 1950
-Wire Wire Line
 	6375 1950 6375 2050
 Wire Wire Line
 	6375 2050 5800 2050
 Wire Wire Line
-	7300 3200 7300 2150
+	7300 2950 7300 2150
 Connection ~ 7300 2150
 Wire Wire Line
@@
 	7100 2050 6450 2050
 Wire Wire Line
-	3800 2350 4750 2350
-Wire Wire Line
 	4750 2050 4150 2050
 Wire Wire Line
 	4150 2050 4150 1950
 Wire Wire Line
-	4150 1950 3800 1950
-Wire Wire Line
 	4750 2150 4100 2150
 Wire Wire Line
 	4100 2150 4100 2050
 Wire Wire Line
-	4100 2050 3800 2050
-Wire Wire Line
 	4750 2250 4050 2250
 Wire Wire Line
 	4050 2250 4050 2150
-Wire Wire Line
-	4050 2150 3800 2150
-Wire Wire Line
-	5800 2350 7475 2350
 $Comp
 L power:GND #PWR0101
@@
 $EndComp
 Wire Wire Line
-	7475 2450 7475 2675
+	7600 2675 7475 2675
+Wire Wire Line
+	7475 2675 7475 2800
+$Comp
+L power:GND #PWR0102
+U 1 1 5CFB9AF2
+P 4500 3275
+F 0 "#PWR0102" H 4500 3025 50  0001 C CNN
+F 1 "GND" H 4500 3125 50  0000 C CNN
+F 2 "" H 4500 3275 50  0000 C CNN
+F 3 "" H 4500 3275 50  0000 C CNN
+	1    4500 3275
+	1    0    0    -1
+$EndComp
+Wire Wire Line
+	4500 3275 4500 3100
+Connection ~ 4500 3100
+Wire Wire Line
+	6900 2875 6900 3100
+$Comp
+L Connector:Conn_01x06_Male J1
+U 1 1 5D3478C0
+P 2850 2150
+F 0 "J1" H 2958 2531 50  0000 C CNN
+F 1 "3V3" H 2958 2440 50  0000 C CNN
+F 2 "Pin_Headers:Pin_Header_Straight_1x06" H 2850 2150 50  0001 C CNN
+F 3 "~" H 2850 2150 50  0001 C CNN
+	1    2850 2150
+	1    0    0    -1
+$EndComp
+$Comp
+L Connector:Conn_01x06_Male J2
+U 1 1 5D34A5F6
+P 9075 2250
+F 0 "J2" H 9047 2132 50  0000 R CNN
+F 1 "5V" H 9047 2223 50  0000 R CNN
+F 2 "Pin_Headers:Pin_Header_Straight_1x06" H 9075 2250 50  0001 C CNN
+F 3 "~" H 9075 2250 50  0001 C CNN
+	1    9075 2250
+	-1   0    0    1
+$EndComp
+$Comp
+L Device:LED D1
+U 1 1 5D34F47E
+P 6900 2725
+F 0 "D1" V 6925 2900 50  0000 R CNN
+F 1 "LED" V 6825 2950 50  0000 R CNN
+F 2 "LEDs:LED_1206" H 6900 2725 50  0001 C CNN
+F 3 "~" H 6900 2725 50  0001 C CNN
+	1    6900 2725
+	0    -1   -1   0
+$EndComp
+$Comp
+L Device:LED D2
+U 1 1 5D352BFF
+P 7100 3100
+F 0 "D2" V 6975 3225 50  0000 R CNN
+F 1 "LED" V 6900 3300 50  0000 R CNN
+F 2 "LEDs:LED_1206" H 7100 3100 50  0001 C CNN
+F 3 "~" H 7100 3100 50  0001 C CNN
+	1    7100 3100
+	0    -1   -1   0
+$EndComp
+$Comp
+L Device:LED D3
+U 1 1 5D3539F8
+P 7300 3100
+F 0 "D3" V 7200 2975 50  0000 R CNN
+F 1 "LED" V 7100 2975 50  0000 R CNN
+F 2 "LEDs:LED_1206" H 7300 3100 50  0001 C CNN
+F 3 "~" H 7300 3100 50  0001 C CNN
+	1    7300 3100
+	0    -1   -1   0
+$EndComp
+$Comp
+L speculatrix_power:LM1117 LM1
+U 1 1 5D349286
+P 5300 1450
+F 0 "LM1" H 5225 1897 60  0000 C CNN
+F 1 "LM1117" H 5225 1791 60  0000 C CNN
+F 2 "TO_SOT_Packages_SMD:SOT-223" H 5300 1450 60  0001 C CNN
+F 3 "" H 5300 1450 60  0000 C CNN
+	1    5300 1450
+	1    0    0    -1
+$EndComp
+$Comp
+L speculatrix_power:TXB0104D_PW IC1
+U 1 1 5D349C51
+P 5300 2350
+F 0 "IC1" H 5275 3087 60  0000 C CNN
+F 1 "TXB0104D_PW" H 5275 2981 60  0000 C CNN
+F 2 "Housings_SOIC:SOIC-14_3.9x8.7mm_Pitch1.27mm" H 5550 1950 60  0001 C CNN
+F 3 "" H 5550 1950 60  0000 C CNN
+	1    5300 2350
+	1    0    0    -1
+$EndComp
 $Comp
 L power:PWR_FLAG #FLG0101
@@
 $EndComp
 Wire Wire Line
-	7600 2675 7475 2675
+	7475 2450 7475 2675
 Connection ~ 7475 2675
-Wire Wire Line
-	7475 2675 7475 2800
-$Comp
-L power:GND #PWR0102
-U 1 1 5CFB9AF2
-P 4500 3275
-F 0 "#PWR0102" H 4500 3025 50  0001 C CNN
-F 1 "GND" H 4500 3125 50  0000 C CNN
-F 2 "" H 4500 3275 50  0000 C CNN
-F 3 "" H 4500 3275 50  0000 C CNN
-	1    4500 3275
-	1    0    0    -1
-$EndComp
-Wire Wire Line
-	4500 3275 4500 3100
-Connection ~ 4500 3100
+$Comp
+L Connector:Conn_01x06_Male J5
+U 1 1 5D3505EC
+P 8400 2750
+F 0 "J5" V 8554 2362 50  0000 R CNN
+F 1 "5V_test" V 8463 2362 50  0000 R CNN
+F 2 "Pin_Headers:Pin_Header_Straight_1x06" H 8400 2750 50  0001 C CNN
+F 3 "~" H 8400 2750 50  0001 C CNN
+	1    8400 2750
+	0    -1   -1   0
+$EndComp
+Wire Wire Line
+	3575 2350 4750 2350
+Wire Wire Line
+	3050 2350 3575 2350
+Connection ~ 3575 2350
+Wire Wire Line
+	3575 2600 3575 2350
+Wire Wire Line
+	3675 2450 3800 2450
+Wire Wire Line
+	3050 2450 3675 2450
+Connection ~ 3675 2450
+Wire Wire Line
+	3675 2600 3675 2450
+$Comp
+L Connector:Conn_01x02_Male J4
+U 1 1 5D35A966
+P 3575 2800
+F 0 "J4" V 3729 2612 50  0000 R CNN
+F 1 "3V3_test2" V 3500 2825 50  0000 R CNN
+F 2 "Pin_Headers:Pin_Header_Straight_1x02" H 3575 2800 50  0001 C CNN
+F 3 "~" H 3575 2800 50  0001 C CNN
+	1    3575 2800
+	0    -1   -1   0
+$EndComp
+Wire Wire Line
+	3375 2150 3050 2150
+Wire Wire Line
+	4050 2150 3375 2150
+Connection ~ 3375 2150
+Wire Wire Line
+	3375 2600 3375 2150
+Wire Wire Line
+	3275 2050 3050 2050
+Wire Wire Line
+	4100 2050 3275 2050
+Connection ~ 3275 2050
+Wire Wire Line
+	3275 2600 3275 2050
+Wire Wire Line
+	3175 1950 3050 1950
+Wire Wire Line
+	4150 1950 3175 1950
+Connection ~ 3175 1950
+Wire Wire Line
+	3175 2600 3175 1950
+$Comp
+L Connector:Conn_01x03_Male J3
+U 1 1 5D35B94D
+P 3275 2800
+F 0 "J3" V 3425 3100 50  0000 R CNN
+F 1 "3V3_test1" V 3200 3225 50  0000 R CNN
+F 2 "Pin_Headers:Pin_Header_Straight_1x03" H 3275 2800 50  0001 C CNN
+F 3 "~" H 3275 2800 50  0001 C CNN
+	1    3275 2800
+	0    -1   -1   0
+$EndComp
+Wire Wire Line
+	6375 1950 8700 1950
+Wire Wire Line
+	7100 2050 8600 2050
+Wire Wire Line
+	7300 2150 8500 2150
+Wire Wire Line
+	7225 2250 8400 2250
+Wire Wire Line
+	5800 2350 8300 2350
+Wire Wire Line
+	7475 2450 8200 2450
+Wire Wire Line
+	8200 2550 8200 2450
+Connection ~ 8200 2450
+Wire Wire Line
+	8200 2450 8875 2450
+Wire Wire Line
+	8300 2550 8300 2350
+Connection ~ 8300 2350
+Wire Wire Line
+	8300 2350 8875 2350
+Wire Wire Line
+	8400 2550 8400 2250
+Connection ~ 8400 2250
+Wire Wire Line
+	8400 2250 8875 2250
+Wire Wire Line
+	8500 2550 8500 2150
+Connection ~ 8500 2150
+Wire Wire Line
+	8500 2150 8875 2150
+Wire Wire Line
+	8600 2550 8600 2050
+Connection ~ 8600 2050
+Wire Wire Line
+	8600 2050 8875 2050
+Wire Wire Line
+	8700 2550 8700 1950
+Connection ~ 8700 1950
+Wire Wire Line
+	8700 1950 8875 1950
 $EndSCHEMATC
